Commit message: Updated URDF for simulator controls.

File: stembot_description/urdf/frame.urdf.xacro (robot description, xacro)
@@ -1,5 +1,14 @@
 <?xml version="1.0"?>
 <robot xmlns:xacro="http://ros.org/wiki/xacro">
-  <!-- Links -->
+  <!--             -->
+  <!-- Frame Links -->
+  <!--             -->
+  <link name="base_link">
+    <inertial>
+      <origin xyz="0.0019 0 -.0006" rpy="0 0 0" />
+      <mass value="${mass}" />
+      <xacro:insert_block name="moment" />
+    </inertial>
+  </link>
   <link name="frame_crossbar">
     <visual>
@@ -57,5 +66,7 @@
   <xacro:lower prefix="port" reflect="-1" />
   <xacro:lower prefix="stbd" reflect="1" />
-  <!-- Joints -->
+  <!--              -->
+  <!-- Frame Joints -->
+  <!--              -->
   <joint name="frame_crossbar" type="fixed">
     <origin xyz="${frame_mount_x} 0 -${frame_mount_z}" rpy="0 0 0" />

File: stembot_description/urdf/housing.urdf.xacro (robot description, xacro)
@@ -1,5 +1,7 @@
 <?xml version="1.0"?>
 <robot xmlns:xacro="http://ros.org/wiki/xacro">
-  <!-- Links -->
+  <!--               -->
+  <!-- Housing Links -->
+  <!--               -->
   <link name="main_housing">
     <visual>
@@ -50,5 +52,7 @@
   <xacro:tube prefix="inner" radius="${inner_radius}" height="${housing_z+0.0055}" color="DarkGrey" />
   <xacro:tube prefix="outer" radius="${outer_radius}" height="${housing_z+0.0050}" color="Grey" />
-  <!-- Joints -->
+  <!--                -->
+  <!-- Housing Joints -->
+  <!--                -->
   <joint name="base_housing" type="fixed">
     <parent link="base_link" />

File: stembot_description/urdf/material.gazebo.xacro (robot description, xacro)
@@ -1,5 +1,9 @@
 <?xml version="1.0"?>
 <robot name="stembot" xmlns:xacro="http://ros.org/wiki/xacro">
-  <!-- Housing -->
+  <!--                  -->
+  <!-- Gazebo Material  -->
+  <!--                  -->
+  <!--                  -->
+  <!-- Housing          -->
   <gazebo reference="main_housing">
     <material>Gazebo/DarkGrey</material>
@@ -21,5 +25,6 @@
     <material>Gazebo/Grey</material>
   </gazebo>
-  <!-- Rods -->
+  <!--                  -->
+  <!-- Rods             -->
   <xacro:macro name="rod_gazebo" params="prefix postfix">
     <gazebo reference="${prefix}_rod_${postfix}">
@@ -35,5 +40,6 @@
   <xacro:rod_gazebo prefix="aft" postfix="3" />
   <xacro:rod_gazebo prefix="aft" postfix="4" />
-  <!-- Frame -->
+  <!--                  -->
+  <!-- Frame            -->
   <gazebo reference="frame_crossbar">
     <material>Gazebo/FlatBlack</material>

File: stembot_description/urdf/rods.urdf.xacro (robot description, xacro)
@@ -1,5 +1,7 @@
 <?xml version="1.0"?>
 <robot xmlns:xacro="http://ros.org/wiki/xacro">
-  <!-- Links -->
+  <!--            -->
+  <!-- Rod Links  -->
+  <!--            -->
   <xacro:macro name="fwd_rod" params="postfix">
     <link name="fwd_rod_${postfix}">
@@ -32,5 +34,7 @@
   <xacro:aft_rod postfix="3" />
   <xacro:aft_rod postfix="4" />
-  <!-- Joints -->
+  <!--             -->
+  <!-- Rod Joints  -->
+  <!--             -->
   <xacro:macro name="fwd_rod_position" params="postfix reflect_y reflect_z">
     <joint name="fwd_rod_${postfix}" type="fixed">

File: stembot_description/urdf/stembot.urdf.xacro (robot description, xacro)
@@ -1,23 +1,58 @@
 <?xml version="1.0"?>
 <robot name="stembot" xmlns:xacro="http://ros.org/wiki/xacro">
-  <link name="base_link">
-    <inertial>
-      <origin xyz="0.0019 0 -.0006" rpy="0 0 0" />
-      <mass value="${mass}" />
-      <xacro:insert_block name="moment" />
-    </inertial>
-  </link>
-  <xacro:include filename="properties.urdf.xacro" />
   <xacro:include filename="housing.urdf.xacro" />
   <xacro:include filename="rods.urdf.xacro" />
   <xacro:include filename="frame.urdf.xacro" />
-  <gazebo>
-    <plugin name="BuoyancyPlugin" filename="libBuoyancyPlugin.so">
-      <link name="base_link">
-        <center_of_volume>0 0 0</center_of_volume>
-        <volume>${volume}</volume>
-      </link>
-    </plugin>
-  </gazebo>
+  <xacro:include filename="material.urdf.xacro" />
+  <xacro:include filename="control.gazebo.xacro" />
   <xacro:include filename="material.gazebo.xacro" />
+  <xacro:property name="M_PI" value="3.1415926535897931" />
+  <xacro:property name="volume" value="0.0032" />
+  <xacro:property name="volume_x" value="0.0000" />
+  <xacro:property name="volume_y" value="0.0000" />
+  <xacro:property name="volume_z" value="0.0000" />
+  <xacro:property name="mass" value="3.4255" />
+  <xacro:property name="mass_x" value="0.0019" />
+  <xacro:property name="mass_y" value="0.0000" />
+  <xacro:property name="mass_z" value="-.0006" />
+  <xacro:property name="moment">
+    <inertia ixx="0.0012" ixy="0.0000" ixz="0.0000"
+             iyy="0.0322" iyz="0.0000"
+             izz="0.0380"/>
+  </xacro:property>
+  <xacro:property name="housing_x" value="0.2381" />
+  <xacro:property name="housing_y" value="0.1270" />
+  <xacro:property name="housing_z" value="0.0762" />
+  <xacro:property name="endcap_x" value="0.0254" />
+  <xacro:property name="endcap_y" value="0.1524" />
+  <xacro:property name="endcap_z" value="0.0953" />
+  <xacro:property name="fwd_plate_x" value="0.0095" />
+  <xacro:property name="fwd_plate_y" value="0.0699" />
+  <xacro:property name="fwd_plate_z" value="0.0575" />
+  <xacro:property name="aft_plate_x" value="0.0064" />
+  <xacro:property name="aft_plate_y" value="0.0508" />
+  <xacro:property name="aft_plate_z" value="0.0381" />
+  <xacro:property name="inner_radius" value="0.0381" />
+  <xacro:property name="outer_radius" value="0.0445" />
+  <xacro:property name="tube_x" value="0.0508" />
+  <xacro:property name="tube_y" value="0.0000" />
+  <xacro:property name="tube_z" value="0.0000" />
+  <xacro:property name="rod_radius" value="0.0064" />
+  <xacro:property name="fwd_rod_ln" value="0.1064" />
+  <xacro:property name="aft_rod_ln" value="0.1254" />
+  <xacro:property name="frame_mount_x" value="${(housing_x-frame_thickness)/2-fwd_rod_ln}" />
+  <xacro:property name="frame_mount_y" value="0.0375" />
+  <xacro:property name="frame_mount_z" value="0.0500" />
+  <xacro:property name="frame_plate_x" value="0.0445" />
+  <xacro:property name="frame_plate_y" value="0.0318" />
+  <xacro:property name="frame_plate_z" value="0.0064" />
+  <xacro:property name="frame_crossbar" value="0.0982" />
+  <xacro:property name="frame_upper" value="0.0550" />
+  <xacro:property name="frame_lower" value="0.0750" />
+  <xacro:property name="frame_thickness" value="0.0064" />
+  <xacro:property name="frame_angle" value="0.5943" />
+  <xacro:property name="frame_radius" value="0.0159" />
+  <xacro:property name="cylinder_fix">
+    <origin xyz="0 0 0" rpy="0 ${M_PI/2} 0" />
+  </xacro:property>
 </robot>
